File: LEDBoard_4x4_HD/LEDBoard_4x4_HD.sch (KiCad schematic (older format))
At the start: 17 parts, among them U1 TLC5957

Commit message: LEDBoard parts positioned & routing started
Parts:
- added C1: 0.1uF, Capacitor_SMD:C_0603_1608Metric_Pad1.05x0.95mm_HandSolder, symbol Device:C
- added J1: power, Connector_PinHeader_2.54mm:PinHeader_1x02_P2.54mm_Vertical, symbol Connector_Generic:Conn_01x02
- added J2: data, Connector_PinHeader_2.54mm:PinHeader_1x05_P2.54mm_Vertical, symbol Connector_Generic:Conn_01x05
- added R1: 7.5KOhm 0.1%, Resistor_SMD:R_0603_1608Metric_Pad1.05x0.95mm_HandSolder, symbol Device:R
- D_0x0, D_0x1, D_0x2, D_0x3, D_1x0, D_1x1, D_1x2, D_1x3, D_2x0, D_2x1, D_2x2, D_2x3, D_3x0, D_3x1, D_3x2, D_3x3: footprint LEDs_SMD_NICHIA:LED_RGB_0706_1816Metric_ROHM__VeryNarow -> LEDs_SMD_NICHIA:LED_RGB_0706_1816Metric_ROHM_ThermalVias
- U1: footprint Package_DFN_QFN:QFN-56-1EP_8x8mm_P0.5mm_EP4.5x5.2mm_ThermalVias -> Package_DFN_QFN:QFN-56-1EP_8x8mm_P0.5mm_EP5.6x5.6mm_ThermalVias; symbol Driver_LED:TLC5957 -> Driver_LED:TLC5957RTQ
Connections:
- net VCC: now also U1.43 (VCC), C1.2, J1.1 (Pin_1)
- net led_0x0_b: now also U1.10 (OUTB0)
- net led_0x0_g: now also U1.9 (OUTG0)
- net led_0x0_r: now also U1.8 (OUTR0)
- net led_0x1_b: now also U1.22 (OUTB4)
- net led_0x1_g: now also U1.21 (OUTG4)
- net led_0x1_r: now also U1.20 (OUTR4)
- net led_0x2_b: now also U1.38 (OUTB8)
- net led_0x2_g: now also U1.37 (OUTG8)
- net led_0x2_r: now also U1.36 (OUTR8)
- net led_0x3_b: now also U1.52 (OUTB12)
- net led_0x3_g: now also U1.51 (OUTG12)
- net led_0x3_r: now also U1.50 (OUTR12)
- net led_1x0_b: now also U1.13 (OUTB1)
- net led_1x0_g: now also U1.12 (OUTG1)
- net led_1x0_r: now also U1.11 (OUTR1)
- net led_1x1_b: now also U1.25 (OUTB5)
- net led_1x1_g: now also U1.24 (OUTG5)
- net led_1x1_r: now also U1.23 (OUTR5)
- net led_1x2_b: now also U1.41 (OUTB9)
- net led_1x2_g: now also U1.40 (OUTG9)
- net led_1x2_r: now also U1.39 (OUTR9)
- net led_1x3_b: now also U1.55 (OUTB13)
- net led_1x3_g: now also U1.54 (OUTG13)
- net led_1x3_r: now also U1.53 (OUTR13)
- net led_2x0_b: now also U1.16 (OUTB2)
- net led_2x0_g: now also U1.15 (OUTG2)
- net led_2x0_r: now also U1.14 (OUTR2)
- net led_2x1_b: now also U1.32 (OUTB6)
- net led_2x1_g: now also U1.31 (OUTG6)
- net led_2x1_r: now also U1.30 (OUTR6)
- net led_2x2_b: now also U1.46 (OUTB10)
- net led_2x2_g: now also U1.45 (OUTG10)
- net led_2x2_r: now also U1.44 (OUTR10)
- net led_2x3_b: now also U1.4 (OUTB14)
- net led_2x3_g: now also U1.3 (OUTG14)
- net led_2x3_r: now also U1.2 (OUTR14)
- net led_3x0_b: now also U1.19 (OUTB3)
- net led_3x0_g: now also U1.18 (OUTG3)
- net led_3x0_r: now also U1.17 (OUTR3)
- net led_3x1_b: now also U1.35 (OUTB7)
- net led_3x1_g: now also U1.34 (OUTG7)
- net led_3x1_r: now also U1.33 (OUTR7)
- net led_3x2_b: now also U1.49 (OUTB11)
- net led_3x2_g: now also U1.48 (OUTG11)
- net led_3x2_r: now also U1.47 (OUTR11)
- net led_3x3_b: now also U1.7 (OUTB15)
- net led_3x3_g: now also U1.6 (OUTG15)
- net led_3x3_r: now also U1.5 (OUTR15)
- new net GCLK: J2.1 (Pin_1), U1.29 (GCLK)
- new net GND: C1.1, J1.2 (Pin_2), R1.1, U1.56 (IREFGND), U1.57 (GND)
- new net IREF: R1.2, U1.1 (IREF)
- new net LAT: J2.2 (Pin_2), U1.27 (LAT)
- new net SCLK: J2.3 (Pin_3), U1.28 (SCLK)
- new net SIN: J2.4 (Pin_4), U1.26 (SIN)
- new net SOUT: J2.5 (Pin_5), U1.42 (SOUT)
Other:
- note added: "1.209V/25mA*154.5 = 7.49kOhm\n154.5 / 7,5kOhm * 1.209V = 24.9 mA\n25mA / 1.209V * ?kOhm = 154.5"
- note added: "BC → Gain → Iolc(@7.5kOhm)\n0h → 000 → 20.0 → 3.2mA (recommend)\n1h → 001 → 39.5 → 6.4mA\n2h → 010 → 58.6 → 9.5mA\n3h → 011 → 80.9 → 13.0mA\n4h → 100 → 100.0 → 16.1mA (default)\n5h → 101 → 113.3 → 18.3mA\n6h → 110 → 141.6 → 22.8mA\n7h → 111 → 154.5 → 24.9mA"

Commit message: first routing done
Parts:
- added C2, C3: 0.1uF, Capacitor_SMD:C_0603_1608Metric_Pad1.05x0.95mm_HandSolder, symbol Device:C
Connections:
- net GND: now also C2.1, C3.1
- net LAT: now also J2.3 (Pin_3); no longer J2.2 (Pin_2)
- net SCLK: now also J2.2 (Pin_2); no longer J2.3 (Pin_3)
- net VCC: now also C2.2, C3.2
Changed lines of the file:
@@
 Text Label 2900 4650 0    50   ~ 0
 GCLK
+Text Label 2900 4850 0    50   ~ 0
+LAT
 Text Label 2900 4750 0    50   ~ 0
-LAT
-Text Label 2900 4850 0    50   ~ 0
 SCLK
 Text Label 2900 4950 0    50   ~ 0
@@
 	1    0    0    -1
 $EndComp
+$Comp
+L Device:C C2
+U 1 1 5BD17E11
+P 3950 1800
+F 0 "C2" H 3836 1754 50  0000 R CNN
+F 1 "0.1uF" H 3836 1845 50  0000 R CNN
+F 2 "Capacitor_SMD:C_0603_1608Metric_Pad1.05x0.95mm_HandSolder" H 3988 1650 50  0001 C CNN
+F 3 "~" H 3950 1800 50  0001 C CNN
+	1    3950 1800
+	1    0    0    1
+$EndComp
+$Comp
+L power:GND #PWR0124
+U 1 1 5BD17E17
+P 3950 1950
+F 0 "#PWR0124" H 3950 1700 50  0001 C CNN
+F 1 "GND" H 3955 1777 50  0000 C CNN
+F 2 "" H 3950 1950 50  0001 C CNN
+F 3 "" H 3950 1950 50  0001 C CNN
+	1    3950 1950
+	1    0    0    -1
+$EndComp
+$Comp
+L power:VCC #PWR0125
+U 1 1 5BD17E1D
+P 3950 1650
+F 0 "#PWR0125" H 3950 1500 50  0001 C CNN
+F 1 "VCC" H 3967 1823 50  0000 C CNN
+F 2 "" H 3950 1650 50  0001 C CNN
+F 3 "" H 3950 1650 50  0001 C CNN
+	1    3950 1650
+	1    0    0    -1
+$EndComp
+$Comp
+L Device:C C3
+U 1 1 5BD1A8DB
+P 3200 1800
+F 0 "C3" H 3086 1754 50  0000 R CNN
+F 1 "0.1uF" H 3086 1845 50  0000 R CNN
+F 2 "Capacitor_SMD:C_0603_1608Metric_Pad1.05x0.95mm_HandSolder" H 3238 1650 50  0001 C CNN
+F 3 "~" H 3200 1800 50  0001 C CNN
+	1    3200 1800
+	1    0    0    1
+$EndComp
+$Comp
+L power:GND #PWR0126
+U 1 1 5BD1A8E1
+P 3200 1950
+F 0 "#PWR0126" H 3200 1700 50  0001 C CNN
+F 1 "GND" H 3205 1777 50  0000 C CNN
+F 2 "" H 3200 1950 50  0001 C CNN
+F 3 "" H 3200 1950 50  0001 C CNN
+	1    3200 1950
+	1    0    0    -1
+$EndComp
+$Comp
+L power:VCC #PWR0127
+U 1 1 5BD1A8E7
+P 3200 1650
+F 0 "#PWR0127" H 3200 1500 50  0001 C CNN
+F 1 "VCC" H 3217 1823 50  0000 C CNN
+F 2 "" H 3200 1650 50  0001 C CNN
+F 3 "" H 3200 1650 50  0001 C CNN
+	1    3200 1650
+	1    0    0    -1
+$EndComp

Commit message: updated pcb fixed some small things added capacitor
Parts:
- added C4: 47uF 6.3V, Capacitor_SMD:C_0603_1608Metric_Pad1.05x0.95mm_HandSolder, symbol Device:C
- C1: value 0.1uF -> 47uF 6.3V
Connections:
- net GND: now also C4.1
- net VCC: now also C4.2
Other:
- moved on the sheet: C3
Changed lines of the file:
@@
 P 3950 950
 F 0 "C1" H 3836 904 50  0000 R CNN
-F 1 "0.1uF" H 3836 995 50  0000 R CNN
+F 1 "47uF 6.3V" H 3836 995 50  0000 R CNN
 F 2 "Capacitor_SMD:C_0603_1608Metric_Pad1.05x0.95mm_HandSolder" H 3988 800 50  0001 C CNN
 F 3 "~" H 3950 950 50  0001 C CNN
@@
 L Device:C C3
 U 1 1 5BD1A8DB
-P 3200 1800
-F 0 "C3" H 3086 1754 50  0000 R CNN
-F 1 "0.1uF" H 3086 1845 50  0000 R CNN
-F 2 "Capacitor_SMD:C_0603_1608Metric_Pad1.05x0.95mm_HandSolder" H 3238 1650 50  0001 C CNN
-F 3 "~" H 3200 1800 50  0001 C CNN
-	1    3200 1800
+P 8650 5150
+F 0 "C3" H 8536 5104 50  0000 R CNN
+F 1 "0.1uF" H 8536 5195 50  0000 R CNN
+F 2 "Capacitor_SMD:C_0603_1608Metric_Pad1.05x0.95mm_HandSolder" H 8688 5000 50  0001 C CNN
+F 3 "~" H 8650 5150 50  0001 C CNN
+	1    8650 5150
 	1    0    0    1
 $EndComp
@@
 L power:GND #PWR0126
 U 1 1 5BD1A8E1
-P 3200 1950
-F 0 "#PWR0126" H 3200 1700 50  0001 C CNN
-F 1 "GND" H 3205 1777 50  0000 C CNN
-F 2 "" H 3200 1950 50  0001 C CNN
-F 3 "" H 3200 1950 50  0001 C CNN
-	1    3200 1950
+P 8650 5300
+F 0 "#PWR0126" H 8650 5050 50  0001 C CNN
+F 1 "GND" H 8655 5127 50  0000 C CNN
+F 2 "" H 8650 5300 50  0001 C CNN
+F 3 "" H 8650 5300 50  0001 C CNN
+	1    8650 5300
 	1    0    0    -1
 $EndComp
@@
 L power:VCC #PWR0127
 U 1 1 5BD1A8E7
-P 3200 1650
-F 0 "#PWR0127" H 3200 1500 50  0001 C CNN
-F 1 "VCC" H 3217 1823 50  0000 C CNN
-F 2 "" H 3200 1650 50  0001 C CNN
-F 3 "" H 3200 1650 50  0001 C CNN
-	1    3200 1650
+P 8650 5000
+F 0 "#PWR0127" H 8650 4850 50  0001 C CNN
+F 1 "VCC" H 8667 5173 50  0000 C CNN
+F 2 "" H 8650 5000 50  0001 C CNN
+F 3 "" H 8650 5000 50  0001 C CNN
+	1    8650 5000
 	1    0    0    -1
 $EndComp
+$Comp
+L Device:C C4
+U 1 1 5BCD1F67
+P 9400 5150
+F 0 "C4" H 9286 5104 50  0000 R CNN
+F 1 "47uF 6.3V" H 9286 5195 50  0000 R CNN
+F 2 "Capacitor_SMD:C_0603_1608Metric_Pad1.05x0.95mm_HandSolder" H 9438 5000 50  0001 C CNN
+F 3 "~" H 9400 5150 50  0001 C CNN
+	1    9400 5150
+	1    0    0    1
+$EndComp
+$Comp
+L power:GND #PWR0128
+U 1 1 5BCD1F6D
+P 9400 5300
+F 0 "#PWR0128" H 9400 5050 50  0001 C CNN
+F 1 "GND" H 9405 5127 50  0000 C CNN
+F 2 "" H 9400 5300 50  0001 C CNN
+F 3 "" H 9400 5300 50  0001 C CNN
+	1    9400 5300
+	1    0    0    -1
+$EndComp
+$Comp
+L power:VCC #PWR0129
+U 1 1 5BCD1F73
+P 9400 5000
+F 0 "#PWR0129" H 9400 4850 50  0001 C CNN
+F 1 "VCC" H 9417 5173 50  0000 C CNN
+F 2 "" H 9400 5000 50  0001 C CNN
+F 3 "" H 9400 5000 50  0001 C CNN
+	1    9400 5000
+	1    0    0    -1
+$EndComp
