File: LEDBoard_4x4_HD.sch (KiCad schematic (older format))
At the start: 25 parts, among them J1 power, J2 data, J3 power, U1 TLC5957

Commit message: updated component
Connections:
- net IREF: now also U1.1 (IREF)
Other:
- moved on the sheet: R1
Changed lines of the file:
@@
 EESchema Schematic File Version 4
 LIBS:LEDBoard_4x4_HD-cache
-EELAYER 26 0
+EELAYER 29 0
 EELAYER END
 $Descr A4 11693 8268
@@
 L Device:R R1
 U 1 1 5BCD32F7
-P 4500 6550
-F 0 "R1" H 4430 6504 50  0000 R CNN
-F 1 "7.5KOhm 0.1%" H 4430 6595 50  0000 R CNN
-F 2 "Resistor_SMD:R_0603_1608Metric_Pad1.05x0.95mm_HandSolder" V 4430 6550 50  0001 C CNN
-F 3 "~" H 4500 6550 50  0001 C CNN
-	1    4500 6550
+P 4250 6000
+F 0 "R1" H 4180 5954 50  0000 R CNN
+F 1 "7.5KOhm 0.1%" H 4180 6045 50  0000 R CNN
+F 2 "Resistor_SMD:R_0603_1608Metric_Pad1.05x0.95mm_HandSolder" V 4180 6000 50  0001 C CNN
+F 3 "~" H 4250 6000 50  0001 C CNN
+	1    4250 6000
 	1    0    0    1
 $EndComp
-Wire Wire Line
-	4500 6700 4600 6700
 Wire Wire Line
 	4600 6700 4600 6200
@@
 Text Notes 5000 6500 0    30   ~ 0
 1.209V/25mA*154.5 = 7.49kOhm\n154.5 / 7,5kOhm * 1.209V = 24.9 mA\n25mA / 1.209V * ?kOhm = 154.5
-Text Label 4500 6400 1    50   ~ 0
+Text Label 4250 5850 1    50   ~ 0
 IREF
 Wire Wire Line
-	4500 6200 4500 6400
+	4250 5600 4250 5850
 Wire Wire Line
 	4800 6200 4800 6700
@@
 	3250 5550 2900 5550
 Connection ~ 2900 5550
+Wire Wire Line
+	4250 5600 4300 5600
+Wire Wire Line
+	4250 6150 4250 6700
+Wire Wire Line
+	4250 6700 4600 6700
 $EndSCHEMATC
